Commit message: temp - 소스코드 정리 필요

File: urdf/lidar.urdf (robot description, URDF)
Before this commit: robot xycar, 7 links, 6 joints
Links:
- removed link base
- removed link base_link
- added link front_left_60
- added link front_right_60
Joints:
- removed joint base_link_to_base
- removed joint base_to_lidar
- added joint front_to_front_left_60: type fixed, parent front, child front_left_60, origin xyz=-0.0 0.0 0.0 rpy=0.0 0.0 1.04
- added joint front_to_front_right_60: type fixed, parent front, child front_right_60, origin xyz=-0.0 0.0 0.0 rpy=0.0 0.0 -1.04
- joint lidar_to_back: origin xyz=0.1 0.0 0.0 rpy=0.0 0.0 3.14 -> xyz=0.0 0.0 0.0 rpy=0.0 0.0 0.0
- joint lidar_to_front: origin xyz=0.1 0.0 0.0 rpy=0.0 0.0 0 -> xyz=-0.0 0.0 0.0 rpy=0.0 0.0 3.14
- joint lidar_to_left: origin xyz=0.0 -0.1 0.0 rpy=0.0 0.0 -1.57 -> xyz=0.0 0.0 0.0 rpy=0.0 0.0 +1.57
- joint lidar_to_right: origin xyz=0.0 0.1 0.0 rpy=0.0 0.0 +1.57 -> xyz=0.0 -0.0 0.0 rpy=0.0 0.0 -1.57
